File: PCBFinal1/PCB Design.kicad_sch (KiCad schematic)
At the start: 13 parts, among them J1 Screw_Terminal_01x02, J2 Screw_Terminal_01x03, J3 Screw_Terminal_01x03, J4 Screw_Terminal_01x02, J5 Screw_Terminal_01x02, K1 SANYOU_SRD_Form_C, Q1 BC547, U1 DEVKIT_V1_ESP32-WROOM-32

Commit message: Finished with the soil calibrations and first version of the pcb design.
Parts:
- added J6: Screw_Terminal_01x04, TerminalBlock_Phoenix:TerminalBlock_Phoenix_MKDS-1,5-4-5.08_1x04_P5.08mm_Horizontal, symbol Connector:Screw_Terminal_01x04
- added R3: 470, Resistor_THT:R_Axial_DIN0207_L6.3mm_D2.5mm_P7.62mm_Horizontal, symbol Device:R
- added R4: 10k, Resistor_THT:R_Axial_DIN0207_L6.3mm_D2.5mm_P7.62mm_Horizontal, symbol Device:R
Connections:
- net GND: now also J2.3 (Pin_3), J3.1 (Pin_1), J4.1 (Pin_1), U1.18 (D18), U1.GND, J6.3 (Pin_3), R4.1
- net at K1.3: now also J1.1 (Pin_1)
- net at K1.4: no longer J1.1 (Pin_1)
- net at U1.12 (D12): no longer J3.3 (Pin_3)
- net at Q1.2 (B): now also R3.2, R4.2; no longer U1.13 (D13)
- net at U1.19 (D19): now also J4.2 (Pin_2)
- net at J2.1 (Pin_1), J3.2 (Pin_2): now also U1.3V3, J6.4 (Pin_4); no longer U1.20 (3V3)
- net at U1.21 (D21): now also J6.1 (Pin_1)
- net at U1.22 (D22): now also J6.2 (Pin_2)
- net at U1.34 (D34): now also J3.3 (Pin_3)
- new net: R3.1, U1.13 (D13)
Other:
- note added: "- OUT +"
- note added: "GND VCC"
- note added: "HIGH-LEVEL TRIGGERED RELAY MODULE FOR PUMP"
- note added: "VCC GND SCL SDA"
- note added: "VIN GND"
- note removed: "+ OUT -"
- note removed: "LOW-LEVEL TRIGGERED RELAY MODULE FOR PUMP"
